Commit message: Lazor

File: nav_u_generic_description/urdf/macros.urdf.xacro (robot description, xacro)
@@ -55,5 +55,5 @@
     <color rgba="0.400000 0.248690 0.020759 1" />
   </material>
-  <xacro:macro name="sensor" params="dx dy:=0 dz parent:=base_link samples angular_range rate:=12.0 min_dist:=0.12 max_dist:=15.0 stddev:=0.01 type:=sensor_msgs/PointCloud2">
+  <xacro:macro name="lazor" params="dx dy:=0 dz parent:=base_link samples angular_range rate:=12.0 min_dist:=0.12 max_dist:=15.0 stddev:=0.01 type:=sensor_msgs/PointCloud2">
     <link name="sensor">
       <visual>

File: nav_u_robot_generator/templates/robot.urdf.xacro (robot description, xacro)
@@ -3,5 +3,5 @@
   <xacro:include filename="$(find nav_u_generic_description)/urdf/macros.urdf.xacro" />
   <xacro:[SHAPE_MACRO] width="[WIDTH]" height="[HEIGHT]" wheel_radius="[WHEEL_RADIUS]" color="[BODY_COLOR]" wheel_color="[WHEEL_COLOR]"/>
-  <xacro:sensor dx="[SENSOR_OFFSET]" dz="[HEIGHT]" samples="[SENSOR_SAMPLES]" angular_range="${[SENSOR_RANGE] * pi / 180}" stddev="[SENSOR_NOISE]" type="sensor_msgs/[SENSOR_TYPE]" />
+  <xacro:lazor dx="[SENSOR_OFFSET]" dz="[HEIGHT]" samples="[SENSOR_SAMPLES]" angular_range="${[SENSOR_RANGE] * pi / 180}" stddev="[SENSOR_NOISE]" type="sensor_msgs/[SENSOR_TYPE]" />
   <xacro:plugins x_covar="0.000004" y_covar="${0.000004*0.5}" theta_covar="${0.2 * 0.000004}" odom_mult="1.18" />
 </robot>

Commit message: [pre-commit.ci] auto fixes from pre-commit.com hooks
for more information, see https://pre-commit.ci

File: nav_u_generic_description/urdf/macros.urdf.xacro (robot description, xacro)
@@ -2,56 +2,56 @@
 <robot xmlns:xacro="http://ros.org/wiki/xacro" name="nav_u">
   <material name="Grey">
-    <color rgba=".3 .3 .3 1" />
+    <color rgba=".3 .3 .3 1"/>
   </material>
   <material name="DarkGrey">
-    <color rgba=".175 .175 .175 1" />
+    <color rgba=".175 .175 .175 1"/>
   </material>
   <material name="White">
-    <color rgba="1 1 1 1" />
+    <color rgba="1 1 1 1"/>
   </material>
   <material name="FlatBlack">
-    <color rgba="0.1 0.1 0.1 1" />
+    <color rgba="0.1 0.1 0.1 1"/>
   </material>
   <material name="Black">
-    <color rgba="0 0 0 1" />
+    <color rgba="0 0 0 1"/>
   </material>
   <material name="Red">
-    <color rgba="1 0 0 1" />
+    <color rgba="1 0 0 1"/>
   </material>
   <material name="RedBright">
-    <color rgba="0.87 0.26 0.07 1" />
+    <color rgba="0.87 0.26 0.07 1"/>
   </material>
   <material name="Green">
-    <color rgba="0 1 0 1" />
+    <color rgba="0 1 0 1"/>
   </material>
   <material name="Blue">
-    <color rgba="0 0 1 1" />
+    <color rgba="0 0 1 1"/>
   </material>
   <material name="SkyBlue">
-    <color rgba="0.13 0.44 0.70 1" />
+    <color rgba="0.13 0.44 0.70 1"/>
   </material>
   <material name="Yellow">
-    <color rgba="1 1 0 1" />
+    <color rgba="1 1 0 1"/>
   </material>
   <material name="ZincYellow">
-    <color rgba="0.9725 0.9529 0.2078 1" />
+    <color rgba="0.9725 0.9529 0.2078 1"/>
   </material>
   <material name="DarkYellow">
-    <color rgba="0.7 0.7 0 1" />
+    <color rgba="0.7 0.7 0 1"/>
   </material>
   <material name="Purple">
-    <color rgba="1 0 1 1" />
+    <color rgba="1 0 1 1"/>
   </material>
   <material name="Turquoise">
-    <color rgba="0 1 1 1" />
+    <color rgba="0 1 1 1"/>
   </material>
   <material name="Orange">
-    <color rgba="1 0.5088 0.0468 1" />
+    <color rgba="1 0.5088 0.0468 1"/>
   </material>
   <material name="Indigo">
-    <color rgba="0.33 0.0 0.5 1" />
+    <color rgba="0.33 0.0 0.5 1"/>
   </material>
   <material name="Gold">
-    <color rgba="0.400000 0.248690 0.020759 1" />
+    <color rgba="0.400000 0.248690 0.020759 1"/>
   </material>
   <xacro:macro name="sensor" params="dx dy:=0 dz parent:=base_link samples angular_range rate:=12.0 min_dist:=0.12 max_dist:=15.0 stddev:=0.01 type:=sensor_msgs/PointCloud2">
@@ -59,22 +59,22 @@
       <visual>
         <geometry>
-          <cylinder radius="0.025" length="0.03" />
-        </geometry>
-        <material name="DarkGrey" />
-      </visual>
-      <collision>
-        <geometry>
-          <cylinder radius="0.025" length="0.03" />
-        </geometry>
-      </collision>
-      <inertial>
-        <mass value="0.1" />
-        <inertia ixx="1e-3" ixy="0.0" ixz="0.0" iyy="1e-3" iyz="0.0" izz="1e-3" />
+          <cylinder radius="0.025" length="0.03"/>
+        </geometry>
+        <material name="DarkGrey"/>
+      </visual>
+      <collision>
+        <geometry>
+          <cylinder radius="0.025" length="0.03"/>
+        </geometry>
+      </collision>
+      <inertial>
+        <mass value="0.1"/>
+        <inertia ixx="1e-3" ixy="0.0" ixz="0.0" iyy="1e-3" iyz="0.0" izz="1e-3"/>
       </inertial>
     </link>
     <joint name="sensor_joint" type="fixed">
-      <parent link="${parent}" />
-      <child link="sensor" />
-      <origin xyz="${dx} ${dy} ${dz + 0.015}" />
+      <parent link="${parent}"/>
+      <child link="sensor"/>
+      <origin xyz="${dx} ${dy} ${dz + 0.015}"/>
     </joint>
     <gazebo reference="sensor">
@@ -84,5 +84,5 @@
           <ros>
             <argument>~/out:=scan</argument>
-            <namespace />
+            <namespace/>
           </ros>
           <output_type>${type}</output_type>
@@ -136,66 +136,66 @@
     <link name="${prefix}_wheel">
       <visual>
-        <origin xyz="0 ${reflect*width/2} 0" rpy="${pi/2} 0 0" />
-        <geometry>
-          <cylinder radius="${radius}" length="${width}" />
-        </geometry>
-        <material name="${color}" />
-      </visual>
-      <collision>
-        <origin xyz="0 ${reflect*width/2} 0" rpy="${pi/2} 0 0" />
-        <geometry>
-          <cylinder radius="${radius}" length="${width}" />
-        </geometry>
-      </collision>
-      <inertial>
-        <mass value="1" />
-        <inertia ixx="1e-3" ixy="0.0" ixz="0.0" iyy="1e-3" iyz="0.0" izz="1e-3" />
+        <origin xyz="0 ${reflect*width/2} 0" rpy="${pi/2} 0 0"/>
+        <geometry>
+          <cylinder radius="${radius}" length="${width}"/>
+        </geometry>
+        <material name="${color}"/>
+      </visual>
+      <collision>
+        <origin xyz="0 ${reflect*width/2} 0" rpy="${pi/2} 0 0"/>
+        <geometry>
+          <cylinder radius="${radius}" length="${width}"/>
+        </geometry>
+      </collision>
+      <inertial>
+        <mass value="1"/>
+        <inertia ixx="1e-3" ixy="0.0" ixz="0.0" iyy="1e-3" iyz="0.0" izz="1e-3"/>
       </inertial>
     </link>
     <joint name="${prefix}_wheel_joint" type="continuous">
-      <axis xyz="0 1 0" rpy="0 0 0" />
-      <parent link="${parent}" />
-      <child link="${prefix}_wheel" />
-      <origin xyz="${dx} ${reflect*(dy + 0.01)} ${dz}" />
+      <axis xyz="0 1 0" rpy="0 0 0"/>
+      <parent link="${parent}"/>
+      <child link="${prefix}_wheel"/>
+      <origin xyz="${dx} ${reflect*(dy + 0.01)} ${dz}"/>
     </joint>
     <gazebo reference="${prefix}_wheel">
-      <mu1 value="0.0" />
-      <mu2 value="0.0" />
-      <kp value="10000000.0" />
-      <kd value="1.0" />
+      <mu1 value="0.0"/>
+      <mu2 value="0.0"/>
+      <kp value="10000000.0"/>
+      <kd value="1.0"/>
       <material>Gazebo/${color}</material>
     </gazebo>
   </xacro:macro>
   <xacro:macro name="box_robot" params="length width height wheel_radius wheel_width:=0.05 color wheel_color:=Black ">
-    <link name="base_footprint" />
+    <link name="base_footprint"/>
     <joint name="foot_to_base_joint" type="fixed">
-      <parent link="base_footprint" />
-      <child link="base_link" />
-      <origin xyz="0 0 ${wheel_radius}" />
+      <parent link="base_footprint"/>
+      <child link="base_link"/>
+      <origin xyz="0 0 ${wheel_radius}"/>
     </joint>
     <link name="base_link">
       <visual>
         <geometry>
-          <box size="${length} ${width} ${height}" />
-        </geometry>
-        <origin xyz="0 0 ${height/2}" />
-        <material name="${color}" />
-      </visual>
-      <collision>
-        <geometry>
-          <box size="${length} ${width} ${height}" />
-        </geometry>
-        <origin xyz="0 0 ${height/2}" />
-      </collision>
-      <inertial>
-        <mass value="10.0" />
-        <inertia ixx="0.12" ixy="0.0" ixz="0.0" iyy="0.4" iyz="0.0" izz="0.5" />
+          <box size="${length} ${width} ${height}"/>
+        </geometry>
+        <origin xyz="0 0 ${height/2}"/>
+        <material name="${color}"/>
+      </visual>
+      <collision>
+        <geometry>
+          <box size="${length} ${width} ${height}"/>
+        </geometry>
+        <origin xyz="0 0 ${height/2}"/>
+      </collision>
+      <inertial>
+        <mass value="10.0"/>
+        <inertia ixx="0.12" ixy="0.0" ixz="0.0" iyy="0.4" iyz="0.0" izz="0.5"/>
       </inertial>
     </link>
     <gazebo reference="base_link">
-      <mu1 value="0.0" />
-      <mu2 value="0.0" />
-      <kp value="10000000.0" />
-      <kd value="1.0" />
+      <mu1 value="0.0"/>
+      <mu2 value="0.0"/>
+      <kp value="10000000.0"/>
+      <kd value="1.0"/>
       <material>Gazebo/${color}</material>
     </gazebo>
@@ -218,33 +218,33 @@
   </xacro:macro>
   <xacro:macro name="circle_robot" params="width height wheel_radius wheel_width:=0.05 color wheel_color:=Orange">
-    <link name="base_footprint" />
+    <link name="base_footprint"/>
     <joint name="foot_to_base_joint" type="fixed">
-      <parent link="base_footprint" />
-      <child link="base_link" />
-      <origin xyz="0 0 ${wheel_radius}" />
+      <parent link="base_footprint"/>
+      <child link="base_link"/>
+      <origin xyz="0 0 ${wheel_radius}"/>
     </joint>
     <link name="base_link">
       <visual>
         <geometry>
-          <cylinder length="${height}" radius="${width / 2}" />
+          <cylinder length="${height}" radius="${width / 2}"/>
         </geometry>
         <origin xyz="0 0 ${height / 2}"/>
-        <material name="${color}" />
-      </visual>
-      <collision>
-        <geometry>
-          <cylinder length="${height}" radius="${width / 2}" />
-        </geometry>
-      </collision>
-      <inertial>
-        <mass value="10.0" />
-        <inertia ixx="0.12" ixy="0.0" ixz="0.0" iyy="0.4" iyz="0.0" izz="0.5" />
+        <material name="${color}"/>
+      </visual>
+      <collision>
+        <geometry>
+          <cylinder length="${height}" radius="${width / 2}"/>
+        </geometry>
+      </collision>
+      <inertial>
+        <mass value="10.0"/>
+        <inertia ixx="0.12" ixy="0.0" ixz="0.0" iyy="0.4" iyz="0.0" izz="0.5"/>
       </inertial>
     </link>
     <gazebo reference="base_link">
-      <mu1 value="0.0" />
-      <mu2 value="0.0" />
-      <kp value="10000000.0" />
-      <kd value="1.0" />
+      <mu1 value="0.0"/>
+      <mu2 value="0.0"/>
+      <kp value="10000000.0"/>
+      <kd value="1.0"/>
       <material>Gazebo/${color}</material>
     </gazebo>
